File: VFO/hardware/fmosc/fmosc.kicad_pcb (KiCad board)
At the start: 2 copper layers, 50 x 50 mm, 42 parts, among them J1 JST PH, J2 U.FL, J3 JST PH, J4 3670128, Q1 MMBT5179, Q2 MMBT5179, Q3 MMBT5179, Q4 MMBT5179

Commit message: R1 for generating gerber
Parts:
- added C10: 10n, g-cap:C_0603_1608Metric, F.Cu at (98.5, 42.0)
- added C11: 27p, g-cap:C_0603_1608Metric, F.Cu at (96.5, 47.0)
- added C12: 39p, g-cap:C_0603_1608Metric, F.Cu at (99.5, 47.0)
- added C13: 1n, g-cap:C_0603_1608Metric, F.Cu at (99.5, 49.0)
- added C14: 10n, g-cap:C_0603_1608Metric, F.Cu at (89.0, 46.5)
- added C15: 4p, g-cap:C_0603_1608Metric, F.Cu at (108.0, 48.5)
- added C17: 10n, g-cap:C_0603_1608Metric, F.Cu at (103.0, 42.5)
- added C18: 10n, g-cap:C_0603_1608Metric, F.Cu at (115.0, 48.5)
- added C19: 10n, g-cap:C_0603_1608Metric, F.Cu at (108.0, 42.5)
- added D4: 1SV325, g-dio:D_SOD-523, F.Cu at (96.5, 49.0)
- added D5: BB133, g-dio:D_SOD-323, F.Cu at (94.5, 71.5)
- added D6: BB133, g-dio:D_SOD-323, F.Cu at (97.5, 71.5)
- added D7: BB133, g-dio:D_SOD-323, F.Cu at (96.5, 49.0)
- added J5: JST PH, g-con:JST_PH_S2B-PH-SM4-TB_1x02-1MP_P2.00mm_Horizontal, F.Cu at (83.5, 46.5)
- added J7: U.FL, g-con:U.FL_Hirose_U.FL-R-SMT-1_Vertical, F.Cu at (125.0, 49.5)
- added L2: 100n, g-ind:L_Wurth_WE-CAIR-4248, F.Cu at (98.0, 75.0)
- added Q5: MMBT5179, g-SOT:SOT-23-3, F.Cu at (99.0, 44.5)
- added Q6: MMBT5179, g-SOT:SOT-23-3, F.Cu at (110.5, 45.0)
- added Q7: MMBT5179, g-SOT:SOT-23-3, F.Cu at (114.0, 45.0)
- added R1: 18K, g-res:R_0603_1608Metric, F.Cu at (101.5, 42.5)
- added R13: 12K, g-res:R_0603_1608Metric, F.Cu at (95.5, 42.0)
- added R14: 2K, g-res:R_0603_1608Metric, F.Cu at (94.5, 44.5)
- added R15: 100E, g-res:R_0603_1608Metric, F.Cu at (96.0, 44.5)
- added R16: 1K, g-res:R_0603_1608Metric, F.Cu at (108.0, 45.5)
- added R17: 3K9, g-res:R_0603_1608Metric, F.Cu at (109.5, 48.5)
- added R18: 820E, g-res:R_0603_1608Metric, F.Cu at (111.5, 48.5)
- added R19: 180E, g-res:R_0603_1608Metric, F.Cu at (113.0, 48.5)
- added R20: 100K, g-res:R_0603_1608Metric, F.Cu at (91.5, 45.5)
- added R21: 47E, g-res:R_0603_1608Metric, F.Cu at (104.5, 42.5)
- D2, D3: value 1SV324 -> 1SV325; footprint g-dio:D_SOD-323 -> g-dio:D_SOD-523
- L1: value 222n -> 82n; footprint g-ind:L_Wurth_WE-CAIR-5910 -> g-ind:L_Wurth_WE-CAIR-4248
- moved R12 23.5 mm to (122.5, 72.9), turned to 0 degrees
- moved C9 23.0 mm to (125.5, 69.5), turned to 90 degrees
- moved Q4 21.0 mm to (122.5, 69.9), turned to 90 degrees
- moved L1 20.9 mm to (104.0, 46.0)
- moved R11 19.9 mm to (119.0, 72.9), turned to 0 degrees
- moved J2 19.0 mm to (124.5, 66.0), turned to 90 degrees
- moved Q1 18.5 mm to (110.0, 77.0), turned to 180 degrees
- moved R5 17.5 mm to (107.0, 76.5)
- moved C6 17.5 mm to (107.0, 73.5)
- moved R7 17.5 mm to (108.5, 73.5)
- moved C8 17.1 mm to (118.5, 79.7)
- moved Q3 16.9 mm to (119.0, 69.9), turned to 90 degrees
- moved C4 16.4 mm to (102.0, 75.5), turned to -90 degrees
- moved R4 16.0 mm to (107.0, 79.5)
- moved C3 14.7 mm to (101.5, 78.0), turned to 0 degrees
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Connections:
- net /F_OUT renamed /Seiler/F_OUT
- net /F_TUNE renamed /Seiler/F_TUNE
- L1 pad 1: GND -> Net-(Q5-C)
- L1 pad 2: Net-(D3-A) -> Net-(C17-Pad1)
Routing:
- net +5V: track 39.4 -> 97.7 mm
- net Net-(Q5-C): track 0.00 -> 19.0 mm
- net GND: track 17.7 -> 29.7 mm, vias 51 -> 76
- net /Common_Base_Colpitts/F_OUT: track 0.00 -> 9.04 mm
- net Net-(D4-K): track 0.00 -> 7.51 mm
- net Net-(Q1-E): track 6.56 -> 14.0 mm, vias 0 -> 2
- net Net-(Q5-B): track 0.00 -> 7.42 mm
- net Net-(C17-Pad1): track 0.00 -> 6.03 mm
- net Net-(Q6-B): track 0.00 -> 4.48 mm
- net Net-(Q5-E): track 0.00 -> 4.38 mm
- net /Common_Base_Colpitts/F_TUNE: track 0.00 -> 4.19 mm
- net Net-(C11-Pad2): track 0.00 -> 3.65 mm
- net Net-(Q7-E): track 0.00 -> 3.56 mm
- net Net-(Q6-E): track 0.00 -> 3.16 mm
- net Net-(D2-K): track 6.10 -> 8.22 mm
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