File: detector/hardware/fm-detector/fm-detector.kicad_sch (KiCad schematic)
At the start: 15 parts, among them J1 JST PH, J2 U.FL, J4 3.5mm audio socket

Commit message: pulse detector design
Parts:
- C25: Voltage 50V -> 50
Connections:
- net +5V: no longer TP1.1
- net Detector/AF: no longer J4.R, J4.T
- net GND: no longer TP2.1
- new net audio_filter/OUT: J4.R, J4.T
Other:
- removed sheet Locked-oscillator-limiter-discriminator
- removed sheet RF-Frontend
- added sheet IF2_amp (IF2_amp.kicad_sch)
- added sheet audio_filter (audio_filter.kicad_sch)
- moved on the sheet: C25, D1, FD1, FD2, FD3, H1, H2, H3, H4, J1, J2, J4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
