File: detector/hardware/fm-detector/fm-detector.kicad_sch (KiCad schematic)
At the start: 15 parts, among them J1 JST PH, J2 U.FL, J4 3.5mm audio socket

Commit message: PCB-0010-0100 ready for release
Parts:
- added FD4, FD5, FD6: Fiducial, g-no_bom:Fiducial_1mm_Mask2mm, symbol g-no_bom:Fiducial
- added J3, J5, J8: U.FL, g-con:U.FL_Hirose_U.FL-R-SMT-1_Vertical, symbol #gplm:con/CON-0001-0000
Connections:
- net +5V: now also TP1.1
- net GND: now also TP2.1, J3.2 (Ext), J5.2 (Ext), J8.2 (Ext)
- net audio filter 1/OUT: no longer J4.R, J4.T
- net Mixer/IF renamed IF
- new net AUDIO: J4.R, J4.T
- new net LFIN: J3.1 (In)
- new net LFOUT: J5.1 (In)
- new net LO: J8.1 (In)
Other:
- sheet audio_filter renamed audio filter 1
- added sheet Board2board (B2B.kicad_sch)
- added sheet DBM Experiments (DBM-experiments.kicad_sch)
- added sheet audio filter 2 (audio_filter.kicad_sch)
- sheet Detector ports: added PWM_AUDIO; removed AF
- note added: "Audio output"
- title: IF2 Oscillator -> FM Intermediate Frequency module
- moved on the sheet: C25, D1, FD1, FD2, FD3, H1, H2, H3, H4, J1, J2, J4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

Commit message: PBA-0010-01A0 ready for release
Changed lines of the file:
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@@
 		(dnp no)
 		(property "Reference" "J4"
-			(at 168.91 52.07 0)
+			(at 173.99 71.12 0)
 			(show_name no)
 			(do_not_autoplace no)
