File: detector/hardware/fm-detector/lo1.kicad_sch (KiCad schematic)
At the start: 27 parts, among them J5 U.FL, Q1 MMBT3904, Q2 MMBT3904

Commit message: pulse detector design
Parts:
- removed C1, C10, C2, C6: 10n, g-cap:C_0603_1608Metric, symbol #gplm:cap/CAP-0000-0103
- removed C3, C4: 18p, g-cap:C_0603_1608Metric, symbol #gplm:cap/CAP-0000-0180
- removed C5: 220p, g-cap:C_0603_1608Metric, symbol #gplm:cap/CAP-0000-0221
- removed C7: 100n, g-cap:C_0603_1608Metric, symbol #gplm:cap/CAP-0000-0104
- removed C8: 10p, g-cap:C_0603_1608Metric, symbol #gplm:cap/CAP-0000-0100
- removed C9: 82p, g-cap:C_0603_1608Metric, symbol #gplm:cap/CAP-0000-0820
- removed J5: U.FL, g-con:U.FL_Hirose_U.FL-R-SMT-1_Vertical, symbol #gplm:con/CON-0001-0000
- removed L2, L3: 6µ8, g-ind:L_Coilcraft_1008HQ_2520Metric, symbol #gplm:ind/IND-0002-0682
- removed Q1, Q2: MMBT3904, g-SOT:SOT-23-3, symbol #gplm:trs/TRS-0000-0001
- removed R1, R12, R4, R9: 100E, g-res:R_0603_1608Metric, symbol #gplm:res/RES-0000-1000
- removed R2, R7: 4K7, g-res:R_0603_1608Metric, symbol #gplm:res/RES-0000-4701
- removed R3: 2K2, g-res:R_0603_1608Metric, symbol #gplm:res/RES-0000-2201
- removed R5: 1K2, g-res:R_0603_1608Metric, symbol #gplm:res/RES-0000-1201
- removed R6: 22K, g-res:R_0603_1608Metric, symbol #gplm:res/RES-0000-2202
- removed R8: 1K8, g-res:R_0603_1608Metric, symbol #gplm:res/RES-0000-1801
- added C37: 2p - 6p, C_Trimmer_Voltronics_JZ, symbol #gplm:cap/CAP-0004-0060
- added C38, C39: 180p, g-cap:C_0603_1608Metric, symbol #gplm:cap/CAP-0000-0181
- added C40: 47p, g-cap:C_0603_1608Metric, symbol #gplm:cap/CAP-0000-0470
- added C41, C43, C44, C45: 100n, g-cap:C_0603_1608Metric, symbol #gplm:cap/CAP-0000-0104
- added C42: 2p, g-cap:C_0603_1608Metric, symbol #gplm:cap/CAP-0000-0020
- added D6: 1N4148, g-dio:D_SOD-323, symbol #gplm:dio/DIO-0001-0000
- added D7: 3V0, g-dio:D_SOD-523, symbol #gplm:dio/DIO-0002-0000
- added H10, H5, H7, H9: S0991-46R, g-rfm:H_Harwin_S0991-46R, symbol #gplm:rfm/RFM-0000-0010
- added J9: U.FL, g-con:U.FL_Hirose_U.FL-R-SMT-1_Vertical, symbol #gplm:con/CON-0001-0000
- added L8, L9: 47µ, g-ind:L_Murata_LQW32FT_3225, symbol #gplm:ind/IND-0003-0473
- added Q12, Q13: J309, g-SOT:SOT-23-3, symbol #gplm:trs/TRS-0002-0000
- added R38, R41: 100K, g-res:R_0603_1608Metric, symbol #gplm:res/RES-0000-1003
- added R39, R42: 47E, g-res:R_0603_1608Metric, symbol #gplm:res/RES-0000-0470
- added R40: 1K, g-res:R_0603_1608Metric, symbol #gplm:res/RES-0000-1001
- L1: footprint g-ind:L_Coilcraft_1008HQ_2520Metric -> g-ind:L_Murata_LQW32FT_3225; symbol #gplm:ind/IND-0002-0682 -> #gplm:ind/IND-0003-0682; Current 0.2 -> 1.4; IPN IND-0002-0682 -> IND-0003-0682; LCSC C318026 -> C23491588; MPN FHW1008UC6R8JGT -> CWP3230A-6R8M; Manufacturer FH -> BOURNS
Connections:
- net +5V: now also R39.2, R40.2, R42.2
- net GND: now also C37.2, C39.1, C40.2, C41.2, C43.1, C44.2, D7.2 (A), H10.1, H5.1, H7.1, H9.1, J9.2 (Ext), L8.1, L9.1, R38.1, R41.1; no longer L1.1
- net LO: now also C45.2, J9.1 (In)
- net at L1.2: now also C38.2, D6.2 (A), Q12.3 (G), R38.2
- net OSC-OUT: no longer names the net of TP3.1
- net OSC-OUT: now also C38.1, C39.2, C42.1, L8.2, Q12.2 (S)
- new net: C44.1, Q13.1 (D), R42.1
- new net: C45.1, L9.2, Q13.2 (S)
- new net: C42.2, Q13.3 (G), R41.2
- new net: C37.1, C40.1, L1.1
- new net: C43.2, D6.1 (K), D7.1 (K), R40.1
- new net: C41.1, Q12.1 (D), R39.1
Other:
- note added: "./LO/JFET_Clapp/DN_Rutgers.ipynb"
- note removed: "(0.65 Vdc)"
- note removed: "(1.23 Vdc)"
- note removed: "(1.36 Vdc)"
- note removed: "(1.99 Vdc)"
- note removed: "(2.43 Vdc)"
