File: detector/hardware/fm-detector/lo1.kicad_sch (KiCad schematic)
At the start: 27 parts, among them J9 U.FL, Q12 J309, Q13 J309

Commit message: PCB-0010-0100 ready for release
Parts:
- removed J9: U.FL, g-con:U.FL_Hirose_U.FL-R-SMT-1_Vertical, symbol #gplm:con/CON-0001-0000
- added J6: 2118708-2, g-rfm:H_TE_2118708, symbol #gplm:rfm/RFM-0000-0002
- C37: footprint C_Trimmer_Voltronics_JZ -> g-cap:C_Trimmer_Voltronics_JZ
- D7: Current 5.00E-03 -> 0.005
Connections:
- net GND: now also J6.1 (Shield)
Other:
- moved on the sheet: C37, C40, H10, H5, H7, H9
