File: detector/hardware/fm-detector/lold.kicad_sch (KiCad schematic)
At the start: 24 parts, among them J6 U.FL, Q10 MMBT3904, Q11 MMBT3904, Q9 MMBT3904, Y1 10.7M

Commit message: pulse detector design
Parts:
- C26, C27, C28, C29, C31, C32, C33: Voltage 50V -> 50
- C30: Voltage 25V -> 25
