File: detector/hardware/fm-detector/rf-frontend.kicad_sch (KiCad schematic)
At the start: 7 parts, among them J7 U.FL, J8 SMA-RA

Commit message: pulse detector design
Parts:
- C34, C35, C36: Voltage 50V -> 50
- D5: footprint g-dio:D_SOD-323 -> g-dio:D_SOD-523
Changed lines of the file:
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@@
 		(fields_autoplaced yes)
 		(property "Reference" "C36"
-			(at 101.6 59.69 0)
-			(do_not_autoplace yes)
-			(effects
-				(font
-					(size 1.27 1.27)
-				)
+			(at 106.68 58.4199 90)
+			(effects
+				(font
+					(size 1.27 1.27)
+				)
+				(justify right)
 			)
 		)
 		(property "Value" "4p"
-			(at 106.68 59.69 0)
-			(do_not_autoplace yes)
-			(effects
-				(font
-					(size 1.27 1.27)
-				)
+			(at 106.68 60.9599 90)
+			(effects
+				(font
+					(size 1.27 1.27)
+				)
+				(justify right)
 			)
 		)
@@
 			)
 		)
-		(property "Voltage" "50V"
+		(property "Voltage" "50"
 			(at 104.14 60.96 0)
 			(effects
@@
 		(fields_autoplaced yes)
 		(property "Reference" "C34"
-			(at 90.17 48.26 0)
-			(do_not_autoplace yes)
+			(at 90.17 44.45 0)
 			(effects
 				(font
@@
 		)
 		(property "Value" "10p"
-			(at 90.17 53.34 0)
-			(do_not_autoplace yes)
+			(at 90.17 46.99 0)
 			(effects
 				(font
@@
 			)
 		)
-		(property "Voltage" "50V"
+		(property "Voltage" "50"
 			(at 88.9 50.8 0)
 			(effects
@@
 		(fields_autoplaced yes)
 		(property "Reference" "C35"
-			(at 110.49 48.26 0)
-			(do_not_autoplace yes)
+			(at 110.49 44.45 0)
 			(effects
 				(font
@@
 		)
 		(property "Value" "10p"
-			(at 110.49 53.34 0)
-			(do_not_autoplace yes)
+			(at 110.49 46.99 0)
 			(effects
 				(font
@@
 			)
 		)
-		(property "Voltage" "50V"
+		(property "Voltage" "50"
 			(at 109.22 50.8 0)
 			(effects
@@
 		(fields_autoplaced yes)
 		(property "Reference" "L7"
-			(at 93.98 59.69 0)
-			(do_not_autoplace yes)
-			(effects
-				(font
-					(size 1.27 1.27)
-				)
+			(at 97.79 58.4199 90)
+			(effects
+				(font
+					(size 1.27 1.27)
+				)
+				(justify right)
 			)
 		)
 		(property "Value" "180n"
-			(at 97.79 59.69 0)
-			(do_not_autoplace yes)
-			(effects
-				(font
-					(size 1.27 1.27)
-				)
+			(at 97.79 60.9599 90)
+			(effects
+				(font
+					(size 1.27 1.27)
+				)
+				(justify right)
 			)
 		)
@@
 		(dnp no)
 		(fields_autoplaced yes)
-		(property "Reference" "#PWR046"
+		(property "Reference" "#PWR46"
 			(at 78.74 72.39 0)
 			(effects
@@
 					(size 1.27 1.27)
 				)
-				(hide yes)
 			)
 		)
@@
 			(project "fm-detector"
 				(path "/b6194304-53f6-4fe9-b4e3-d7d4346b2089/c6f2bbd6-eb35-43ee-8225-499090b4f694"
-					(reference "#PWR046")
+					(reference "#PWR46")
 					(unit 1)
 				)
@@
 			)
 		)
-		(property "Footprint" "g-dio:D_SOD-323"
+		(property "Footprint" "g-dio:D_SOD-523"
 			(at 79.502 59.69 0)
 			(effects
@@
 		(dnp no)
 		(fields_autoplaced yes)
-		(property "Reference" "#PWR050"
+		(property "Reference" "#PWR50"
 			(at 83.82 72.39 0)
 			(effects
@@
 					(size 1.27 1.27)
 				)
-				(hide yes)
 			)
 		)
@@
 			(project "fm-detector"
 				(path "/b6194304-53f6-4fe9-b4e3-d7d4346b2089/c6f2bbd6-eb35-43ee-8225-499090b4f694"
-					(reference "#PWR050")
+					(reference "#PWR50")
 					(unit 1)
 				)
@@
 		(dnp no)
 		(fields_autoplaced yes)
-		(property "Reference" "#PWR048"
+		(property "Reference" "#PWR48"
 			(at 104.14 72.39 0)
 			(effects
@@
 					(size 1.27 1.27)
 				)
-				(hide yes)
 			)
 		)
@@
 			(project "fm-detector"
 				(path "/b6194304-53f6-4fe9-b4e3-d7d4346b2089/c6f2bbd6-eb35-43ee-8225-499090b4f694"
-					(reference "#PWR048")
+					(reference "#PWR48")
 					(unit 1)
 				)
@@
 		(dnp no)
 		(fields_autoplaced yes)
-		(property "Reference" "#PWR049"
+		(property "Reference" "#PWR49"
 			(at 119.38 72.39 0)
 			(effects
@@
 					(size 1.27 1.27)
 				)
-				(hide yes)
 			)
 		)
@@
 			(project "fm-detector"
 				(path "/b6194304-53f6-4fe9-b4e3-d7d4346b2089/c6f2bbd6-eb35-43ee-8225-499090b4f694"
-					(reference "#PWR049")
+					(reference "#PWR49")
 					(unit 1)
 				)
@@
 		(dnp no)
 		(fields_autoplaced yes)
-		(property "Reference" "#PWR047"
+		(property "Reference" "#PWR47"
 			(at 96.52 72.39 0)
 			(effects
@@
 					(size 1.27 1.27)
 				)
-				(hide yes)
 			)
 		)
@@
 			(project "fm-detector"
 				(path "/b6194304-53f6-4fe9-b4e3-d7d4346b2089/c6f2bbd6-eb35-43ee-8225-499090b4f694"
-					(reference "#PWR047")
+					(reference "#PWR47")
 					(unit 1)
 				)
