File: detector/hardware/fm-detector/B2B.kicad_sch (KiCad schematic)
At the start: 2 parts, among them J11 2x06M, J12 2x06F

Commit message: PBA-0010-01A0 ready for release
Parts:
- J11: LCSC C41370963 -> C3975189
- J12: LCSC C41370963 -> C41397115
Changed lines of the file:
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@@
 			)
 		)
-		(property "LCSC" "C41370963"
+		(property "LCSC" "C3975189"
 			(at 91.44 43.18 0)
 			(hide yes)
@@
 			)
 		)
-		(property "LCSC" "C41370963"
-			(at 91.44 66.04 0)
-			(hide yes)
+		(property "LCSC" "C41397115"
+			(at 91.44 66.04 0)
+			(hide yes)
