File: detector/hardware/fm-detector/DBM_TLine.kicad_sch (KiCad schematic)
At the start: 11 parts, among them J13 U.FL, J14 U.FL, J15 U.FL

Commit message: PBA-0010-01A0 ready for release
Changed lines of the file:
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@@
 		(dnp no)
 		(property "Reference" "D4"
-			(at 93.98 31.75 0)
+			(at 101.6 46.99 0)
 			(show_name no)
 			(do_not_autoplace no)
@@
 		)
 		(property "Value" "BAT15-099R"
-			(at 101.6 46.99 0)
+			(at 101.6 31.75 0)
 			(show_name no)
 			(do_not_autoplace no)
@@
 		(dnp no)
 		(fields_autoplaced yes)
-		(property "Reference" "#PWR076"
+		(property "Reference" "#PWR76"
 			(at 144.78 44.45 0)
 			(hide yes)
@@
 			(project "fm-detector"
 				(path "/b6194304-53f6-4fe9-b4e3-d7d4346b2089/467c2634-fe48-47e5-adb8-da867342ddb1/75d2aed5-2303-4a94-8697-ac591b60a742"
-					(reference "#PWR076")
+					(reference "#PWR76")
 					(unit 1)
 				)
@@
 		(dnp no)
 		(fields_autoplaced yes)
-		(property "Reference" "#PWR074"
+		(property "Reference" "#PWR74"
 			(at 81.28 74.93 0)
 			(hide yes)
@@
 			(project "fm-detector"
 				(path "/b6194304-53f6-4fe9-b4e3-d7d4346b2089/467c2634-fe48-47e5-adb8-da867342ddb1/75d2aed5-2303-4a94-8697-ac591b60a742"
-					(reference "#PWR074")
+					(reference "#PWR74")
 					(unit 1)
 				)
@@
 		(dnp no)
 		(fields_autoplaced yes)
-		(property "Reference" "#PWR072"
+		(property "Reference" "#PWR72"
 			(at 45.72 44.45 0)
 			(hide yes)
@@
 			(project "fm-detector"
 				(path "/b6194304-53f6-4fe9-b4e3-d7d4346b2089/467c2634-fe48-47e5-adb8-da867342ddb1/75d2aed5-2303-4a94-8697-ac591b60a742"
-					(reference "#PWR072")
+					(reference "#PWR72")
 					(unit 1)
 				)
