File: detector/hardware/fm-detector/IF2_amp.kicad_sch (KiCad schematic)
At the start: 16 parts, among them J5 U.FL, J7 U.FL, Q1 MMBT3904

Commit message: PCB-0010-0100 ready for release
Parts:
- removed J5, J7: U.FL, g-con:U.FL_Hirose_U.FL-R-SMT-1_Vertical, symbol #gplm:con/CON-0001-0000
Other:
- sheet IF2_amp_stage renamed IF2_amp_stage_I
- sheet IF2_amp_stage1 renamed IF2_amp_stage_II
- sheet IF2_amp_stage2 renamed IF2_amp_stage_III
