File: detector/hardware/fm-detector/IF2_amp_sub.kicad_sch (KiCad schematic)
At the start: 7 parts, among them Q2 MMBT3904

Commit message: PCB-0010-0100 ready for release
Parts:
- renumbered C7 to C10, C8 to C19, C9 to C20, Q2 to Q8, R7 to R12, R5 to R8, R6 to R9
