File: detector/hardware/fm-detector/mixer.kicad_sch (KiCad schematic)
At the start: 11 parts, among them J3 U.FL, Q3 BSS138

Commit message: PCB-0010-0100 ready for release
Parts:
- removed J3: U.FL, g-con:U.FL_Hirose_U.FL-R-SMT-1_Vertical, symbol #gplm:con/CON-0001-0000
Other:
- title: IF2 Mixer -> Simple FET switching mixer
